Commit message: 1st working version

File: urdf/jaska_robot.xacro (robot description, xacro)
@@ -30,8 +30,5 @@
     <xacro:property name="rocker_mesh_rpy" value="${M_PI/2} 0 ${M_PI}" />
     <xacro:property name="bogie_mesh_rpy" value="${M_PI/2} 0 0" />
-    <xacro:property name="wheel_mesh_rpy" value="0 0 0" />
-    <xacro:property name="sensor_mount_mesh_rpy" value="0 0 0" />
-    <xacro:property name="lidar_mesh_rpy" value="0 0 0" />
-    <xacro:property name="camera_mesh_rpy" value="0 0 0" />
+    <xacro:property name="wheel_mesh_rpy" value="${M_PI/2} 0 0" />
     <!-- Mesh scale adjustments (typically 0.001 for mm to meters conversion) -->
     <xacro:property name="trunk_mesh_scale" value="0.09 0.09 0.09" />
@@ -220,5 +217,5 @@
         <link name="${wheel_prefix}_wheel">
             <visual>
-                <origin xyz="0 0 0" rpy="${M_PI/2} 0 ${wheel_mesh_rpy}"/>
+                <origin xyz="0 0 0" rpy="${wheel_mesh_rpy}"/>
                 <geometry>
                     <mesh filename="package://jaska_description/meshes/wheel.stl" scale="${wheel_mesh_scale}"/>
@@ -304,5 +301,5 @@
         parent_link="right_bogie"
         wheel_offset_x="${-bogie_length/2 - 0.050}"
-        wheel_offset_y="-0.050"
+        wheel_offset_y="-0.060"
         wheel_offset_z="-0.110" />
     <!-- Differential drive constraint: synchronize left and right wheels -->
@@ -314,5 +311,5 @@
     <link name="sensor_mount_base">
         <visual>
-            <origin xyz="0 0 0" rpy="${sensor_mount_mesh_rpy}" />
+            <origin xyz="0 0 0" rpy="0 0 0" />
             <geometry>
                 <mesh filename="package://jaska_description/meshes/lidar_and_camera_mount.stl" scale="${sensor_mount_mesh_scale}"/>
@@ -348,5 +345,5 @@
     <link name="unitree_lidar_link">
         <visual>
-            <origin xyz="-0.037 -0.037 -0.025" rpy="${lidar_mesh_rpy}" />
+            <origin xyz="-0.037 -0.037 -0.025" rpy="0 0 0" />
             <geometry>
                 <!-- Use actual Unitree L2 mesh from local meshes directory -->
@@ -397,5 +394,5 @@
     <link name="zed_camera_center">
         <visual>
-            <origin xyz="0 0 0" rpy="${camera_mesh_rpy}"/>
+            <origin xyz="0 0 0" rpy="0 0 0"/>
             <geometry>
                 <mesh filename="package://jaska_description/meshes/zedx.stl" scale="${camera_mesh_scale}"/>

Commit message: Add Isaac Sim support

File: urdf/jaska_robot.xacro (robot description, xacro)
@@ -374,12 +374,50 @@
         <origin xyz="0.010 0.042 0.135" rpy="0 ${sensor_mount_angle} 0"/>
     </joint>
-    <!-- Unitree L2 Lidar Optical Frame -->
-    <link name="unitree_lidar_optical_frame"/>
+    <!-- Unitree L2 Lidar Optical Frame (matches real hardware frame name) -->
+    <link name="unilidar_lidar"/>
     <joint name="unitree_lidar_optical_joint" type="fixed">
         <parent link="unitree_lidar_link"/>
-        <child link="unitree_lidar_optical_frame"/>
+        <child link="unilidar_lidar"/>
         <!-- Lidar optical frame at sensor center -->
         <origin xyz="0 0 0.030" rpy="0 0 0"/>
     </joint>
+    <!-- Gazebo 3D Lidar Sensor Plugin for Unitree L2 -->
+    <gazebo reference="unitree_lidar_link">
+        <material>Gazebo/Black</material>
+        <sensor name="unitree_l2_lidar" type="gpu_lidar">
+            <pose>0 0 0.030 0 0 0</pose>
+            <always_on>true</always_on>
+            <visualize>true</visualize>
+            <update_rate>10</update_rate>
+            <topic>unilidar/cloud</topic>
+            <gz_frame_id>unilidar_lidar</gz_frame_id>
+            <lidar>
+                <scan>
+                    <horizontal>
+                        <samples>1800</samples>
+                        <min_angle>-3.14159</min_angle>
+                        <max_angle>3.14159</max_angle>
+                        <resolution>1.0</resolution>
+                    </horizontal>
+                    <vertical>
+                        <samples>32</samples>
+                        <min_angle>-0.1047</min_angle>  <!-- -6 degrees (downward) -->
+                        <max_angle>1.5708</max_angle>   <!-- +90 degrees (upward dome) -->
+                        <resolution>1.0</resolution>
+                    </vertical>
+                </scan>
+                <range>
+                    <min>0.1</min>
+                    <max>30.0</max>  <!-- Unitree L2 max range -->
+                    <resolution>0.01</resolution>
+                </range>
+                <noise>
+                    <type>gaussian</type>
+                    <mean>0.0</mean>
+                    <stddev>0.01</stddev>
+                </noise>
+            </lidar>
+        </sensor>
+    </gazebo>
     <!-- ============================================== -->
     <!-- ZED X CAMERA - Simplified from ZED ROS2 Wrapper -->
